File: Shield1/Shield1.kicad_sch (KiCad schematic)
At the start: 31 parts

Commit message: v0.2 circuit is ready
Parts:
- removed J? (x23): Conn_01x01_Male, symbol Connector:Conn_01x01_Male
- removed J?: USB_C_Receptacle, symbol Connector:USB_C_Receptacle
- removed U? (x2): TPS2513, Package_TO_SOT_SMD:SOT-23-6, symbol Interface_USB:TPS2513
- added C? (x2): C, Capacitor_SMD:C_0402_1005Metric, symbol Device:C
- added J? (x28): Conn_01x01_Male, symbol Connector:Conn_01x01_Male
- added U? (x2): TPS2553, symbol Shield1:TPS2553
- added X?: USB_C_24pins, symbol Shield1:USB_C_24pins
Connections:
- net Earth: now also J?.1 (Pin_1), X?.S1 (SHIELD)
- net GND1: now also C?.2, R?.2, C?.1, J?.1 (Pin_1), J?.1 (Pin_1), J?.1 (Pin_1), J?.1 (Pin_1), U?.2 (GND), X?.A1 (GND), X?.B12 (GND)
- net GND2: now also C?.2, R?.2, C?.1, J?.1 (Pin_1), J?.1 (Pin_1), J?.1 (Pin_1), J?.1 (Pin_1), U?.2 (GND), X?.A12 (GND), X?.B1 (GND)
- net VBUS: now also C?.2, U?.6 (OUT), X?.A4 (VBUS), X?.B9 (VBUS)
- net VDD: now also C?.2, U?.6 (OUT), X?.A9 (VBUS), X?.B4 (VBUS)
- net at R?.1: now also U?.5 (Ilim) (x2)
- net at C?.1: now also J?.1 (Pin_1), U?.1 (IN) (x2)
- new net: J?.1 (Pin_1), U?.3 (EN) (x2)
- new net: J?.1 (Pin_1), X?.A5 (CC1)
- new net: J?.1 (Pin_1), X?.B11 (RX1+)
- new net: J?.1 (Pin_1), X?.B3 (TX2-)
- new net: J?.1 (Pin_1), X?.B10 (RX1-)
- new net: J?.1 (Pin_1), X?.A8 (SBU1)
- new net: J?.1 (Pin_1), X?.B5 (CC2)
- new net: J?.1 (Pin_1), U?.4 (OC) (x2)
- new net: J?.1 (Pin_1), X?.A2 (TX1+)
- new net: J?.1 (Pin_1), X?.A7 (D-), X?.B7 (D-)
- new net: J?.1 (Pin_1), X?.A3 (TX1-)
- new net: J?.1 (Pin_1), X?.B8 (SBU2)
- new net: J?.1 (Pin_1), X?.A11 (RX2+)
- new net: J?.1 (Pin_1), X?.A6 (D+), X?.B6 (D+)
- new net: J?.1 (Pin_1), X?.A10 (RX2-)
- new net: J?.1 (Pin_1), X?.B2 (TX2+)
Other:
- moved on the sheet: C?, J?, R?
