File: Shield1/_autosave-Shield1.kicad_sch (KiCad schematic)
At the start: 24 parts, among them J1 Conn_01x01_Male, J10 Conn_01x01_Male, J11 Conn_01x01_Male, J12 Conn_01x01_Male, J13 Conn_01x01_Male, J14 Conn_01x01_Male, J15 Conn_01x01_Male, J16 Conn_01x01_Male, J17 Conn_01x01_Male, J18 Conn_01x01_Male, J19 Conn_01x01_Male, J2 Conn_01x01_Male, J3 Conn_01x01_Male, J4 Conn_01x01_Male, J5 Conn_01x01_Male, J6 Conn_01x01_Male, J7 Conn_01x01_Male, J8 Conn_01x01_Male, J9 Conn_01x01_Male, X1 USB_C_24pins

Commit message: v0.3 Cшксгше was reduced, initial decpmposition has been completed
Parts:
- gave numbers to parts that had none: 2
- renumbered C1 to C2, C2 to C3
Changed lines of the file:
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@@
   (symbol (lib_id "Device:C") (at 93.98 55.88 180) (unit 1)
     (in_bom yes) (on_board yes) (fields_autoplaced)
-    (property "Reference" "C?" (id 0) (at 90.17 57.1501 0)
+    (property "Reference" "C4" (id 0) (at 90.17 57.1501 0)
       (effects (font (size 1.27 1.27)) (justify left))
     )
@@
   (symbol (lib_id "Device:C") (at 144.78 30.48 270) (unit 1)
     (in_bom yes) (on_board yes) (fields_autoplaced)
-    (property "Reference" "C?" (id 0) (at 146.0501 34.29 0)
+    (property "Reference" "C1" (id 0) (at 146.0501 34.29 0)
       (effects (font (size 1.27 1.27)) (justify left))
     )
@@
   (symbol (lib_id "Device:C") (at 104.14 54.61 180) (unit 1)
     (in_bom yes) (on_board yes) (fields_autoplaced)
-    (property "Reference" "C2" (id 0) (at 100.33 55.8801 0)
+    (property "Reference" "C3" (id 0) (at 100.33 55.8801 0)
       (effects (font (size 1.27 1.27)) (justify left))
     )
@@
   (symbol (lib_id "Device:C") (at 142.24 38.1 270) (unit 1)
     (in_bom yes) (on_board yes) (fields_autoplaced)
-    (property "Reference" "C1" (id 0) (at 143.5101 41.91 0)
+    (property "Reference" "C2" (id 0) (at 143.5101 41.91 0)
       (effects (font (size 1.27 1.27)) (justify left))
     )
@@
       (reference "#PWR07") (unit 1) (value "GND2") (footprint "")
     )
+    (path "/0808c325-8330-401e-a38b-e2f753ef1f13"
+      (reference "C1") (unit 1) (value "C") (footprint "Capacitor_SMD:C_0402_1005Metric")
+    )
     (path "/fe78c5b9-6d8e-4bb7-98df-a03bb92646f5"
-      (reference "C1") (unit 1) (value "C") (footprint "Capacitor_SMD:C_0402_1005Metric")
+      (reference "C2") (unit 1) (value "C") (footprint "Capacitor_SMD:C_0402_1005Metric")
     )
     (path "/fb2e9001-db82-43dc-8fa8-fcc0e82a26bc"
-      (reference "C2") (unit 1) (value "C") (footprint "Capacitor_SMD:C_0402_1005Metric")
+      (reference "C3") (unit 1) (value "C") (footprint "Capacitor_SMD:C_0402_1005Metric")
     )
     (path "/002bd37c-2cdf-42fa-9224-e629dce93a31"
-      (reference "C?") (unit 1) (value "C") (footprint "Capacitor_SMD:C_0402_1005Metric")
-    )
-    (path "/0808c325-8330-401e-a38b-e2f753ef1f13"
-      (reference "C?") (unit 1) (value "C") (footprint "Capacitor_SMD:C_0402_1005Metric")
+      (reference "C4") (unit 1) (value "C") (footprint "Capacitor_SMD:C_0402_1005Metric")
     )
     (path "/1f4d8215-5efe-4f79-b16f-06aa692013a9"
